File: Riverhawk-3D-Printer.kicad_sch (KiCad schematic)
At the start: 0 parts

Commit message: Select microcontroller and stepper motor drivers
Parts:
- added A1, A2, A3, A4: Pololu_Breakout_A4988, Module:Pololu_Breakout-16_15.2x20.3mm, symbol Driver_Motor:Pololu_Breakout_A4988
- added U1: STM32G431KBUx, Package_DFN_QFN:QFN-32-1EP_5x5mm_P0.5mm_EP3.45x3.45mm, symbol MCU_ST_STM32G4:STM32G431KBUx
Connections:
- new net: U1.16 (VSS), U1.32 (VSS), U1.33 (VSS)
Other:
- title: (none) -> Riverhawk 3D Printer motherboard
